File: hardware/digital_submodule/bluetooth-daq-digital-submodule/bluetooth-daq-digital-submodule.kicad_sch (KiCad schematic)
At the start: 142 parts, among them J1 MCU I/F, J2 Digital Inputs, J3 Digital Outputs, J4 Communication I/F, J5 RS-485 I/F, U1 74HC595, U2 74HC595, U3 74HC165, U4 74HC165, U5 24LC1025, U6 SN75176AD, U7 CD4053B, U8 CD4053B

Commit message: Performed first successful initial PCB routing
Connections:
- net +3V3 renamed 3V3
