File: hardware/analog_submodule/analog_submodule/analog_submodule.kicad_sch (KiCad schematic)
At the start: 213 parts, among them J1 HVIN1, J10 HSADC in, J2 HVIN2, J3 CIN1, J4 CIN2, J5 LVIN+, J6 LVIN-, J7 RES_THERM, J8 AOUT, J9 MCU I/F, Q1 BSS138, Q2 BSS138, Q3 BSS138, Q4 BSS138, U1 AMS1117-5.0, U10 CD4051B, U100 LM6171D, U11 TL084, U12 TL084, U13 TLV9002IDR, U2 CD4051B, U3 CD4051B, U4 CD4051B, U5 CD4051B, U6 TLV9004IDR, U7 ADS131M02IPWR, U8 DAC101C081CIMK, U9 LM6171D, X1 ASV-xxxMHz

Commit message: Completed PCB design for analog submodule
Parts:
- added J11: HSADC in, Connector_PinHeader_2.54mm:PinHeader_1x04_P2.54mm_Vertical, symbol Connector_Generic:Conn_01x04
Connections:
- net AOUT0-: now also J8.2 (Pin_2); no longer J8.8 (Pin_8)
- net AOUT1+: now also J8.3 (Pin_3); no longer J8.2 (Pin_2)
- net AOUT1-: now also J8.4 (Pin_4); no longer J8.7 (Pin_7)
- net AOUT2+: now also J8.5 (Pin_5); no longer J8.3 (Pin_3)
- net AOUT3+: now also J8.7 (Pin_7); no longer J8.4 (Pin_4)
- net AOUT3-: now also J8.8 (Pin_8); no longer J8.5 (Pin_5)
- net GND: now also J9.12 (Pin_12), J9.13 (Pin_13), J11.3 (Pin_3), J11.4 (Pin_4); no longer Q2.1 (G), Q3.1 (G), R113.2, R114.2
- net HSADC0: now also J11.1 (Pin_1); no longer J9.13 (Pin_13)
- net HSADC1: now also J11.2 (Pin_2); no longer J9.12 (Pin_12)
- new net: Q3.1 (G), R114.2
- new net: Q2.1 (G), R113.2
